Commit message: feat(trirotor): add trirotor controller and task configurations, update .gitignore

File: resources/robots/tiltrotor/trirotor.urdf (robot description, URDF)
Before this commit: robot multirotor, 7 links, 6 joints
Links:
- removed link arm_motor_0
- removed link arm_motor_1
- removed link arm_motor_2
- added link connecting_link_motor_0
- added link connecting_link_motor_1
- added link connecting_link_motor_2
- link base_link: mass 0.321 -> 0.221
Joints:
- removed joint base_link_to_arm_motor_0
- removed joint base_link_to_arm_motor_1
- removed joint base_link_to_arm_motor_2
- removed joint base_link_to_motor_0
- removed joint base_link_to_motor_1
- removed joint base_link_to_motor_2
- added joint base_link_to_connecting_link_0: type revolute, parent base_link, child connecting_link_motor_0, origin xyz=0.2 -0.22 0.0 rpy=0.0 0.0 0.0, axis 0 1 0, limit lower=-0.785398 upper=0.785398 effort=20.0 velocity=10.0
- added joint base_link_to_connecting_link_1: type revolute, parent base_link, child connecting_link_motor_1, origin xyz=0.2 0.22 0.0 rpy=0.0 0.0 0.0, axis 0 1 0, limit lower=-0.785398 upper=0.785398 effort=20.0 velocity=10.0
- added joint base_link_to_connecting_link_2: type revolute, parent base_link, child connecting_link_motor_2, origin xyz=-0.43 0.0 0.0 rpy=0.0 0.0 0.0, axis 0 1 0, limit lower=-0.785398 upper=0.785398 effort=20.0 velocity=10.0
- added joint connecting_link_to_motor_0: type fixed, parent connecting_link_motor_0, child motor_0, origin xyz=0 0 0 rpy=0.0 0.0 0.0
- added joint connecting_link_to_motor_1: type fixed, parent connecting_link_motor_1, child motor_1, origin xyz=0 0 0 rpy=0.0 0.0 0.0
- added joint connecting_link_to_motor_2: type fixed, parent connecting_link_motor_2, child motor_2, origin xyz=0 0 0 rpy=0.0 0.0 0.0

Commit message: feat: prepare sim2real align the motor and dynamics

File: resources/robots/tiltrotor/trirotor.urdf (robot description, URDF)
Before this commit: robot multirotor, 7 links, 6 joints
Links:
- link base_link: mass 0.221 -> 2.9
- link motor_0: mass 0.013 -> 0.05
- link motor_1: mass 0.013 -> 0.05
- link motor_2: mass 0.013 -> 0.05

Commit message: real urdf config

File: resources/robots/tiltrotor/trirotor.urdf (robot description, URDF)
Before this commit: robot multirotor, 7 links, 6 joints
Joints:
- joint base_link_to_connecting_link_0: origin xyz=0.2 -0.22 0.0 rpy=0.0 0.0 0.0 -> xyz=0.35 0.42 0.325 rpy=0.0 0.0 0.0
- joint base_link_to_connecting_link_1: origin xyz=0.2 0.22 0.0 rpy=0.0 0.0 0.0 -> xyz=0.35 -0.42 0.300 rpy=0.0 0.0 0.0
- joint base_link_to_connecting_link_2: origin xyz=-0.43 0.0 0.0 rpy=0.0 0.0 0.0 -> xyz=-1.08 0 0.1 rpy=0.0 0.0 0.0

Commit message: feat: sim2real M3 param

File: resources/robots/tiltrotor/trirotor.urdf (robot description, URDF)
Before this commit: robot multirotor, 7 links, 6 joints
Links:
- link base_link: mass 2.9 -> 3.1
